File: FPCBs/Battery/Battery.kicad_sch (KiCad schematic)
At the start: 6 parts

Commit message: Add pad mask
Parts:
- C1, C2: footprint Capacitor_SMD:C_0201_0603Metric -> Leica-G9ii:R_2x1mm
- Connector_Battery1: renamed from Power_Connector_Battery1; footprint Leica-G9ii:Power_Connector_Battery -> Leica-G9ii:Connector_Battery
- F1, R1: footprint Resistor_SMD:R_0201_0603Metric -> Leica-G9ii:R_2x1mm
- FPC_Power1: renamed from Power_Connector_Camera1; footprint Leica-G9ii:Power_Connector_Camera -> Leica-G9ii:FPC_Power
Changed lines of the file:
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@@
 (kicad_sch
-	(version 20231120)
+	(version 20250114)
 	(generator "eeschema")
-	(generator_version "8.0")
+	(generator_version "9.0")
 	(paper "A4")
 	(junction
@@
 			)
 		)
-		(property "Footprint" "Capacitor_SMD:C_0201_0603Metric"
+		(property "Footprint" "Leica-G9ii:R_2x1mm"
 			(at 125.4252 69.85 0)
 			(effects
@@
 			)
 		)
-		(property "Footprint" "Capacitor_SMD:C_0201_0603Metric"
+		(property "Footprint" "Leica-G9ii:R_2x1mm"
 			(at 135.5852 69.85 0)
 			(effects
@@
 			)
 		)
-		(property "Footprint" "Resistor_SMD:R_0201_0603Metric"
+		(property "Footprint" "Leica-G9ii:R_2x1mm"
 			(at 144.78 71.628 90)
 			(effects
@@
 			)
 		)
-		(property "Footprint" "Resistor_SMD:R_0201_0603Metric"
+		(property "Footprint" "Leica-G9ii:R_2x1mm"
 			(at 114.3 69.088 90)
 			(effects
@@
 		(dnp no)
 		(fields_autoplaced yes)
-		(property "Reference" "Power_Connector_Battery1"
+		(property "Reference" "Connector_Battery1"
 			(at 175.26 73.0249 0)
 			(effects
@@
 			)
 		)
-		(property "Footprint" "Leica-G9ii:Power_Connector_Battery"
+		(property "Footprint" "Leica-G9ii:Connector_Battery"
 			(at 166.37 73.66 0)
 			(effects
@@
 			(project ""
 				(path "/49765ffb-117b-4de1-87dd-2e5f7150eecf"
-					(reference "Power_Connector_Battery1")
+					(reference "Connector_Battery1")
 					(unit 1)
 				)
@@
 		(dnp no)
 		(fields_autoplaced yes)
-		(property "Reference" "Power_Connector_Camera1"
+		(property "Reference" "FPC_Power1"
 			(at 92.71 57.15 0)
 			(effects
@@
 			)
 		)
-		(property "Footprint" "Leica-G9ii:Power_Connector_Camera"
+		(property "Footprint" "Leica-G9ii:FPC_Power"
 			(at 92.71 69.85 0)
 			(effects
@@
 			(project ""
 				(path "/49765ffb-117b-4de1-87dd-2e5f7150eecf"
-					(reference "Power_Connector_Camera1")
+					(reference "FPC_Power1")
 					(unit 1)
 				)
@@
 		)
 	)
+	(embedded_fonts no)
 )
