File: FPCBs/USBC/USBC_90deg.kicad_pcb (KiCad board)
At the start: 2 copper layers, 58.5 x 18.1 mm, 2 parts, among them P1 USB_C_Plug, P2 USB_C_Plug

Commit message: Update USBC
Parts:
- moved P1 78.5 mm to (71.6, 150.0)
Routing:
- net Net-(P1-SHIELD): track 76.5 -> 171.0 mm
- net Net-(P1-D+): track 53.5 -> 80.4 mm
- net Net-(P1-TX1-): track 51.0 -> 77.9 mm
- net Net-(P1-TX1+): track 50.2 -> 77.0 mm
- net Net-(P1-SBU1): track 55.2 -> 82.0 mm
- net Net-(P1-RX1+): track 57.7 -> 84.5 mm
- net Net-(P1-D-): track 54.3 -> 81.2 mm
- net Net-(P1-CC): track 52.7 -> 79.5 mm
- net Net-(P1-VCONN): track 58.5 -> 85.4 mm
- net Net-(P1-SBU2): track 56.0 -> 82.9 mm
- net Net-(P1-RX1-): track 56.8 -> 83.7 mm
- net Net-(P1-VBUS-PadA4): track 51.8 -> 78.7 mm
- net Net-(P1-GND-PadA1): track 49.4 -> 76.2 mm
Other:
- board size 58.5 x 18.1 mm -> 18 x 85.2 mm
