File: FPCBs/USBC/USBC.kicad_pcb (KiCad board)
At the start: 2 copper layers, 11.8 x 60.7 mm, 2 parts, among them P1 USB_C_Plug, P2 USB_C_Plug

Commit message: Fix the usbc extender
Parts:
- P1: value USB_C_Plug -> USB_C_Mainboard; footprint Connector_USB:USB-C-12-Pin-MidMount -> Leica-G9ii:FPC_Mainboard_USBC-12Pins
- P2: value USB_C_Plug -> USB_C_Connector; footprint Connector_USB:USB-C-12-Pin-MidMount -> Leica-G9ii:Connector_USBC-12Pins
- moved P1 78.7 mm to (71.1, 150.0)
- moved P2 61.6 mm to (76.0, 80.0), turned to -90 degrees
Routing:
- net (no net): track 0.00 -> 1063.0 mm
- net Net-(P1-SHIELD): track 115.2 -> 0.00 mm
- net Net-(P1-VCONN): track 52.7 -> 0.00 mm
- net Net-(P1-VBUS-PadA4): track 52.7 -> 0.00 mm
- net Net-(P1-TX1-): track 52.7 -> 0.00 mm
- net Net-(P1-TX1+): track 52.7 -> 0.00 mm
- net Net-(P1-SBU2): track 52.7 -> 0.00 mm
- net Net-(P1-SBU1): track 52.7 -> 0.00 mm
- net Net-(P1-RX1-): track 52.7 -> 0.00 mm
- net Net-(P1-RX1+): track 52.7 -> 0.00 mm
- net Net-(P1-GND-PadA1): track 52.7 -> 0.00 mm
- net Net-(P1-D-): track 52.7 -> 0.00 mm
- net Net-(P1-D+): track 52.7 -> 0.00 mm
- net Net-(P1-CC): track 52.7 -> 0.00 mm
Other:
- board size 11.8 x 60.7 mm -> 16.2 x 77 mm
