File: FPCBs/USBC/USBC.kicad_sch (KiCad schematic)
At the start: 2 parts, among them P1 USB_C_Plug, P2 USB_C_Plug

Commit message: Update to kicad 9
Changed lines of the file:
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@@
 (kicad_sch
-	(version 20231120)
+	(version 20250114)
 	(generator "eeschema")
-	(generator_version "8.0")
+	(generator_version "9.0")
 	(paper "A4")
 	(wire
@@
 		)
 	)
+	(embedded_fonts no)
 )

Commit message: Update USBC
Parts:
- P1, P2: footprint Connector_USB:USB-C-12-Pin-MidMount -> Leica-G9ii:USBC-12Pins
Changed lines of the file:
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@@
 			)
 		)
-		(property "Footprint" "Connector_USB:USB-C-12-Pin-MidMount"
+		(property "Footprint" "Leica-G9ii:USBC-12Pins"
 			(at 77.47 96.52 0)
 			(effects
@@
 			)
 		)
-		(property "Footprint" "Connector_USB:USB-C-12-Pin-MidMount"
+		(property "Footprint" "Leica-G9ii:USBC-12Pins"
 			(at 125.73 96.52 0)
 			(effects

Commit message: Fix the usbc extender
Parts:
- P1: value USB_C_Plug -> USB_C_Mainboard; footprint Leica-G9ii:USBC-12Pins -> Leica-G9ii:FPC_Mainboard_USBC-12Pins
- P2: value USB_C_Plug -> USB_C_Connector; footprint Leica-G9ii:USBC-12Pins -> Leica-G9ii:Connector_USBC-12Pins
Changed lines of the file:
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@@
 			)
 		)
-		(property "Value" "USB_C_Plug"
+		(property "Value" "USB_C_Mainboard"
 			(at 73.66 66.04 0)
 			(effects
@@
 			)
 		)
-		(property "Footprint" "Leica-G9ii:USBC-12Pins"
+		(property "Footprint" "Leica-G9ii:FPC_Mainboard_USBC-12Pins"
 			(at 77.47 96.52 0)
 			(effects
@@
 		(fields_autoplaced yes)
 		(property "Reference" "P2"
-			(at 129.54 63.5 0)
+			(at 140.97 99.0599 0)
 			(effects
 				(font
 					(size 1.27 1.27)
 				)
+				(justify right)
 			)
 		)
-		(property "Value" "USB_C_Plug"
-			(at 129.54 66.04 0)
+		(property "Value" "USB_C_Connector"
+			(at 140.97 101.5999 0)
 			(effects
 				(font
 					(size 1.27 1.27)
 				)
+				(justify right)
 			)
 		)
-		(property "Footprint" "Leica-G9ii:USBC-12Pins"
+		(property "Footprint" "Leica-G9ii:Connector_USBC-12Pins"
 			(at 125.73 96.52 0)
 			(effects
