File: FPCBs/Right/Right.kicad_sch (KiCad schematic)
At the start: 24 parts, among them J1 PCB, J4 shutter+1st_dial, J5 2nd Focus+Shutter, J6 Conn_01x03_Pin, SW1 Mode Dial, SW2 ON/OFF, SW3 Focus+Shutter, SW4 Focus+Shutter, SW6 ON/OFF, U1 SG-105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

Commit message: Add Canon shutter footprint
Parts:
- SW3: footprint Leica-G9ii:Switch_Shutter_1 -> Leica-G9ii:Switch_Shutter_Olympus
- SW4: footprint Leica-G9ii:Switch_Shutter_1 -> Leica-G9ii:Switch_Shutter_Canon
Changed lines of the file:
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@@
 			)
 		)
-		(property "Footprint" "Leica-G9ii:Switch_Shutter_1"
+		(property "Footprint" "Leica-G9ii:Switch_Shutter_Olympus"
 			(at 243.84 102.87 0)
 			(effects
@@
 			)
 		)
-		(property "Footprint" "Leica-G9ii:Switch_Shutter_1"
+		(property "Footprint" "Leica-G9ii:Switch_Shutter_Canon"
 			(at 158.75 105.41 0)
 			(effects
