File: FPCBs/Back/Back.kicad_sch (KiCad schematic)
At the start: 28 parts, among them J1 To PCB, J2 To Front, J3 Front, J4 EVF_SENSOR, J5 From LCD, J6 To Right, SW1 MENU/SET, SW10 -+-, SW11 PLAY, SW12 BACK_WHEEL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

Commit message: Fix connectors
Connections:
- net at J3.2 (Pin_2): now also SW13.3 (A); no longer SW13.2 (C)
- net at J3.3 (Pin_3): now also SW13.2 (C); no longer SW13.3 (A)
Other:
- note added: "COM"
- note added: "LVF"
- note added: "M"
- note added: "PLAY"
- note added: "S"
- note added: "S 1-3 C 1-- M 1-2"
- note removed: "S 1-2 C 1-- M 1-3"
Changed lines of the file:
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@@
 	(generator_version "9.0")
 	(paper "A4")
-	(text "S 1-2\nC 1--\nM 1-3"
+	(text "PLAY"
 		(exclude_from_sim no)
-		(at 275.082 131.064 0)
+		(at 98.298 99.314 0)
+		(effects
+			(font
+				(size 1.27 1.27)
+			)
+		)
+	)
+	(text "S"
+		(exclude_from_sim no)
+		(at 74.93 123.444 0)
+		(effects
+			(font
+				(size 1.27 1.27)
+			)
+		)
+	)
+	(text "COM"
+		(exclude_from_sim no)
+		(at 98.044 96.774 0)
+		(effects
+			(font
+				(size 1.27 1.27)
+			)
+		)
+	)
+	(text "S 1-3\nC 1--\nM 1-2"
+		(exclude_from_sim no)
+		(at 271.78 131.064 0)
+		(effects
+			(font
+				(size 1.27 1.27)
+			)
+		)
+	)
+	(text "M"
+		(exclude_from_sim no)
+		(at 74.93 120.904 0)
+		(effects
+			(font
+				(size 1.27 1.27)
+			)
+		)
+	)
+	(text "LVF"
+		(exclude_from_sim no)
+		(at 97.79 101.854 0)
 		(effects
 			(font
@@
 	(wire
 		(pts
-			(xy 269.24 128.27) (xy 265.43 128.27)
-		)
-		(stroke
-			(width 0)
-			(type default)
-		)
-	)
-	(wire
-		(pts
 			(xy 172.72 107.95) (xy 114.3 107.95)
 		)
@@
 	(wire
 		(pts
+			(xy 266.7 128.27) (xy 265.43 128.27)
+		)
+		(stroke
+			(width 0)
+			(type default)
+		)
+	)
+	(wire
+		(pts
 			(xy 88.9 146.05) (xy 88.9 154.94)
 		)
@@
 	(wire
 		(pts
-			(xy 233.68 133.35) (xy 242.57 133.35)
+			(xy 233.68 133.35) (xy 243.84 133.35)
 		)
 		(stroke
@@
 	(wire
 		(pts
-			(xy 240.03 138.43) (xy 269.24 138.43)
+			(xy 266.7 133.35) (xy 265.43 133.35)
 		)
 		(stroke
@@
 	(wire
 		(pts
-			(xy 240.03 135.89) (xy 240.03 138.43)
-		)
-		(stroke
-			(width 0)
-			(type default)
-		)
-	)
-	(wire
-		(pts
 			(xy 215.9 96.52) (xy 214.63 96.52)
 		)
@@
 	(wire
 		(pts
+			(xy 266.7 133.35) (xy 266.7 135.89)
+		)
+		(stroke
+			(width 0)
+			(type default)
+		)
+	)
+	(wire
+		(pts
 			(xy 163.83 77.47) (xy 172.72 77.47)
 		)
@@
 	(wire
 		(pts
-			(xy 242.57 135.89) (xy 265.43 135.89)
+			(xy 243.84 119.38) (xy 266.7 119.38)
 		)
 		(stroke
@@
 	(wire
 		(pts
-			(xy 233.68 135.89) (xy 240.03 135.89)
+			(xy 233.68 135.89) (xy 266.7 135.89)
 		)
 		(stroke
@@
 	(wire
 		(pts
-			(xy 269.24 138.43) (xy 269.24 128.27)
-		)
-		(stroke
-			(width 0)
-			(type default)
-		)
-	)
-	(wire
-		(pts
 			(xy 144.78 57.15) (xy 147.32 57.15)
 		)
@@
 	(wire
 		(pts
+			(xy 266.7 119.38) (xy 266.7 128.27)
+		)
+		(stroke
+			(width 0)
+			(type default)
+		)
+	)
+	(wire
+		(pts
 			(xy 82.55 123.19) (xy 106.68 123.19)
 		)
@@
 	(wire
 		(pts
-			(xy 265.43 135.89) (xy 265.43 133.35)
-		)
-		(stroke
-			(width 0)
-			(type default)
-		)
-	)
-	(wire
-		(pts
 			(xy 233.68 154.94) (xy 266.7 154.94)
 		)
@@
 	(wire
 		(pts
-			(xy 242.57 133.35) (xy 242.57 135.89)
+			(xy 243.84 133.35) (xy 243.84 119.38)
 		)
 		(stroke
@@
 		(on_board yes)
 		(dnp no)
-		(fields_autoplaced yes)
 		(property "Reference" "J5"
-			(at 96.52 101.5999 0)
+			(at 92.456 89.662 0)
 			(effects
 				(font
@@
 		)
 		(property "Value" "From LCD"
-			(at 96.52 104.1399 0)
-			(effects
-				(font
+			(at 90.17 92.456 0)
+			(effects
+				(font
