File: FPCBs/Left/Left.kicad_pcb (KiCad board)
At the start: 2 copper layers, 46.9 x 13.4 mm, 7 parts, among them J1 To PCB, SW1 SW_Rotary_1x6_MP

Commit message: Fix left fpcb
Parts:
- R1: value 1.8K -> 1.7K; footprint Leica-G9ii:R_2x1mm -> Leica-G9ii:R_0603
- R2: value 2.8K -> 2.7K; footprint Leica-G9ii:R_2x1mm -> Leica-G9ii:R_0603
- R3: value 4.8K -> 4.7K; footprint Leica-G9ii:R_2x1mm -> Leica-G9ii:R_0603
- R4: value 8K -> 8.2K; footprint Leica-G9ii:R_2x1mm -> Leica-G9ii:R_0603
- R5: value R -> 22K; footprint Leica-G9ii:R_2x1mm -> Leica-G9ii:R_0603
- moved J1 20.7 mm to (167.6, 91.1)
Connections:
- R1 pad 1: Net-(J1-Pin_1) -> Net-(J1-Pin_2)
- SW1 pad 1: Net-(J1-Pin_1) -> Net-(J1-Pin_2)
- SW1 pad 7: Net-(J1-Pin_2) -> Net-(J1-Pin_1)
Routing:
- net Net-(J1-Pin_1): track 36.9 -> 68.8 mm
- net Net-(J1-Pin_2): track 49.0 -> 58.1 mm
- net Net-(R4-Pad2): track 4.97 -> 4.41 mm
- removed copper zone on B.Cu, net (none)
Other:
- board size 46.9 x 13.4 mm -> 67.4 x 14.7 mm

Commit message: Export new Gerbers and CADs
Other:
- board text added: "JLCJLCJLCJLC"
Changed lines of the file:
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@@
 		(tenting front back)
 		(pcbplotparams
-			(layerselection 0x00000000_00000000_55555555_5755f5ff)
+			(layerselection 0x00000000_00000000_55d55555_5755f5ff)
 			(plot_on_all_layers_selection 0x00000000_00000000_00000000_00000000)
 			(disableapertmacros no)
@@
 		(layer "User.9")
 	)
+	(gr_circle
+		(center 117 98.2)
+		(end 117.8 98.2)
+		(stroke
+			(width 0.1)
+			(type solid)
+		)
+		(fill no)
+		(layer "User.9")
+	)
 	(gr_line
 		(start 168.55 87.55)
@@
 		(layer "User.9")
 	)
+	(gr_circle
+		(center 100 98.2)
+		(end 100.8 98.2)
+		(stroke
+			(width 0.1)
+			(type solid)
+		)
+		(fill no)
+		(layer "User.9")
+	)
 	(gr_line
 		(start 167.55 94.65)
@@
 		(layer "User.9")
 	)
+	(gr_text "JLCJLCJLCJLC"
+		(at 136.41 100.62 0)
+		(layer "F.SilkS")
+		(effects
+			(font
+				(size 1.2 1.2)
+				(thickness 0.25)
+				(bold yes)
+			)
+			(justify bottom)
+		)
+	)
 	(segment
