File: FPCBs/USBC_extender/USBC_extender.kicad_sch (KiCad schematic)
At the start: 2 parts, among them P1 USB_C_Mainboard, P2 USB_C_Connector

Commit message: Export new Gerbers and CADs
Parts:
- P1: footprint Leica-G9ii:FPC_Mainboard_USBC-12Pins -> Leica-G9ii:Connector_USBC-PCB-24Pins; symbol Connector:USB_C_Plug -> Connector:USB_C_Receptacle
- P2: footprint Leica-G9ii:Connector_USBC-12Pins -> Leica-G9ii:Connector_USBC-Receptacle-24Pins; symbol Connector:USB_C_Plug -> Connector:USB_C_Receptacle
Connections:
- net at P1.A1 (GND), P1.A12 (GND), P1.B1 (GND)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: now also P1.S1 (SHIELD), P2.S1 (SHIELD)
- new net: P1.B6 (D+), P2.B6 (D+)
- new net: P1.B7 (D-), P2.B7 (D-)
Changed lines of the file:
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@@
 	(generator_version "9.0")
 	(paper "A4")
+	(junction
+		(at 73.66 139.7)
+		(diameter 0)
+		(color 0 0 0 0)
+	)
+	(junction
+		(at 129.54 139.7)
+		(diameter 0)
+		(color 0 0 0 0)
+	)
 	(wire
 		(pts
@@
 	(wire
 		(pts
+			(xy 88.9 91.44) (xy 114.3 91.44)
+		)
+		(stroke
+			(width 0)
+			(type default)
+		)
+	)
+	(wire
+		(pts
 			(xy 88.9 76.2) (xy 114.3 76.2)
 		)
@@
 	(wire
 		(pts
+			(xy 73.66 139.7) (xy 129.54 139.7)
+		)
+		(stroke
+			(width 0)
+			(type default)
+		)
+	)
+	(wire
+		(pts
 			(xy 88.9 99.06) (xy 114.3 99.06)
 		)
@@
 	(wire
 		(pts
+			(xy 88.9 86.36) (xy 114.3 86.36)
+		)
+		(stroke
+			(width 0)
+			(type default)
+		)
+	)
+	(wire
+		(pts
 			(xy 88.9 78.74) (xy 114.3 78.74)
 		)
@@
 	(wire
 		(pts
-			(xy 137.16 137.16) (xy 137.16 142.24)
+			(xy 137.16 137.16) (xy 137.16 139.7)
 		)
 		(stroke
@@
 	(wire
 		(pts
-			(xy 73.66 139.7) (xy 129.54 139.7)
-		)
-		(stroke
-			(width 0)
-			(type default)
-		)
-	)
-	(wire
-		(pts
-			(xy 66.04 137.16) (xy 66.04 142.24)
+			(xy 66.04 137.16) (xy 66.04 139.7)
 		)
 		(stroke
@@
 	(wire
 		(pts
-			(xy 66.04 142.24) (xy 137.16 142.24)
+			(xy 129.54 139.7) (xy 137.16 139.7)
+		)
+		(stroke
+			(width 0)
+			(type default)
+		)
+	)
+	(wire
+		(pts
+			(xy 66.04 139.7) (xy 73.66 139.7)
 		)
 		(stroke
@@
 	)
 	(symbol
-		(lib_id "Connector:USB_C_Plug")
+		(lib_id "Connector:USB_C_Receptacle")
 		(at 73.66 96.52 0)
 		(unit 1)
@@
 			)
 		)
-		(property "Footprint" "Leica-G9ii:FPC_Mainboard_USBC-12Pins"
+		(property "Footprint" "Leica-G9ii:Connector_USBC-PCB-24Pins"
 			(at 77.47 96.52 0)
 			(effects
@@
 			)
 		)
-		(property "Description" "USB Type-C Plug connector"
+		(property "Description" "USB Full-Featured Type-C Receptacle connector"
 			(at 73.66 96.52 0)
 			(effects
@@
 		)
 		(pin "A1"
+		)
+		(pin "B7"
+		)
+		(pin "B6"
 		)
 		(instances
@@
 	)
 	(symbol
-		(lib_id "Connector:USB_C_Plug")
+		(lib_id "Connector:USB_C_Receptacle")
 		(at 129.54 96.52 0)
 		(mirror y)
@@
 			)
 		)
-		(property "Footprint" "Leica-G9ii:Connector_USBC-12Pins"
+		(property "Footprint" "Leica-G9ii:Connector_USBC-Receptacle-24Pins"
 			(at 125.73 96.52 0)
 			(effects
@@
 			)
 		)
-		(property "Description" "USB Type-C Plug connector"
+		(property "Description" "USB Full-Featured Type-C Receptacle connector"
 			(at 129.54 96.52 0)
 			(effects
@@
 		(pin "A1"
 		)
+		(pin "B7"
+		)
+		(pin "B6"
+		)
 		(instances
